File: hardware/schematic/display_board/display_board_gopro_housing.kicad_pcb (KiCad board)
At the start: 2 copper layers, 52.5 x 43.6 mm, 9 parts, among them J1 Conn_01x04_Pin, SW1 SW_Push, SW2 SW_Push

Commit message: Consolidate display_board/nav_board KiCad files to latest local work
This machine has the most recent hardware design work. Promote the
Rev B design to canonical display_board.kicad_pro/.kicad_sch/.kicad_pcb,
move its matching gerbers/drill files into manufacturing/, track the
gopro-housing variant as a maintained alternate board, and drop the
superseded Rev A files, stale fabrication/ output, and backup zips
(archived locally under a gitignored _archive/ folder rather than
deleted outright). Also brings nav_board's schematic/PCB/manufacturing
files up to date.

Co-Authored-By: Claude Sonnet 5 <noreply@anthropic.com>
Connections:
- A1 pad 10: Net-(A1-IO4/A5) -> unconnected-(A1-IO4/A5-Pad10)
- J1 pad 1: Net-(A1-TX/IO17) -> Net-(A1-RX/IO16)
- J1 pad 2: Net-(A1-RX/IO16) -> Net-(A1-TX/IO17)
- U1 pad 2: Net-(A1-IO4/A5) -> unconnected-(U1-Lite-Pad2)
Routing:
- net Net-(A1-IO4/A5): track 44.5 -> 0.00 mm, vias 1 -> 0
- net Net-(A1-RX/IO16): track 47.5 -> 41.4 mm
- net /3V3: track 62.2 -> 57.6 mm
- net Net-(A1-TX/IO17): track 37.6 -> 37.0 mm
Other:
- board text removed: "Rev B 9/20/26"
